Commit message: diam to radius

File: src/roomba_description/urdf/roomba.urdf (robot description, URDF)
Before this commit: robot roomba, 1 links, 0 joints
Links:
- link base_link: geometry collision cylinder length=0.09225 radius=0.3485/2; visual mesh filename=package://roomba-description/meshes/roomba.dae

Commit message: path change

File: src/roomba_description/urdf/roomba.urdf (robot description, URDF)
Before this commit: robot roomba, 1 links, 0 joints
Links:
- link base_link: geometry collision cylinder length=0.09225 radius=0.3485/2; visual mesh filename=package://roomba_description/meshes/roomba.dae

Commit message: diameter/2

File: src/roomba_description/urdf/roomba.urdf (robot description, URDF)
Before this commit: robot roomba, 1 links, 0 joints
Links:
- link base_link: geometry collision cylinder length=0.09225 radius=0.17425; visual mesh filename=package://roomba_description/meshes/roomba.dae

Commit message: added left wheel

File: src/roomba_description/urdf/roomba.urdf (robot description, URDF)
Before this commit: robot roomba, 1 links, 0 joints
Links:
- added link left_wheel, mass 1; collision cylinder length=0.015 radius=0.036; visual cylinder length=0.015 radius=0.036
Joints:
- added joint left_wheel_joint: type continuous, parent base_link, child left_wheel, origin xyz=0 0 0 rpy=0 1.5708 0, axis 0 1 0

Commit message: added left wheel

File: src/roomba_description/urdf/roomba.urdf (robot description, URDF)
Before this commit: robot roomba, 2 links, 1 joints
Joints:
- joint left_wheel_joint: origin xyz=0 0 0 rpy=0 1.5708 0 -> xyz=0 -0.1175 0 rpy=1.5708 0 0

Commit message: added right wheel

File: src/roomba_description/urdf/roomba.urdf (robot description, URDF)
Before this commit: robot roomba, 2 links, 1 joints
Links:
- added link right_wheel, mass 1; collision cylinder length=0.015 radius=0.036; visual cylinder length=0.015 radius=0.036
Joints:
- added joint right_wheel_joint: type continuous, parent base_link, child right_wheel, origin xyz=0 -0.1175 0 rpy=1.5708 0 0, axis 0 1 0
- joint left_wheel_joint: origin xyz=0 -0.1175 0 rpy=1.5708 0 0 -> xyz=0 0.1175 0 rpy=1.5708 0 0
